Commit message: Address Gazebo hardware review feedback

File: buddy_description/urdf/buddy.urdf.xacro (robot description, xacro)
@@ -39,5 +39,5 @@
   <joint name="caster_joint" type="continuous"><parent link="base_link"/><child link="caster_link"/><origin xyz="-0.18 0 ${-body_height / 2 + 0.02}"/><axis xyz="0 0 1"/></joint>
   <xacro:macro name="sensor_link" params="name xyz rpy *sensor_geometry">
-    <link name="${name}"><visual><origin xyz="${xyz}" rpy="${rpy}"/><geometry><xacro:insert_block name="sensor_geometry"/></geometry><material name="sensor_black"/></visual></link>
+    <link name="${name}"><visual><origin xyz="0 0 0" rpy="0 0 0"/><geometry><xacro:insert_block name="sensor_geometry"/></geometry><material name="sensor_black"/></visual></link>
     <joint name="${name}_joint" type="fixed"><parent link="base_link"/><child link="${name}"/><origin xyz="${xyz}" rpy="${rpy}"/></joint>
   </xacro:macro>

Commit message: fix gazebo command safety contracts

File: buddy_description/urdf/buddy.urdf.xacro (robot description, xacro)
@@ -14,5 +14,4 @@
   <material name="rubber"><color rgba="0.05 0.05 0.05 1"/></material>
   <material name="sensor_black"><color rgba="0.12 0.12 0.12 1"/></material>
-  <link name="base_footprint"/>
   <link name="base_link">
     <inertial><origin xyz="0 0 0"/><mass value="8.0"/>
@@ -21,5 +20,6 @@
     <collision><geometry><box size="${body_length} ${body_width} ${body_height}"/></geometry></collision>
   </link>
-  <joint name="base_footprint_joint" type="fixed"><parent link="base_footprint"/><child link="base_link"/><origin xyz="0 0 ${wheel_radius + body_height / 2}"/></joint>
+  <link name="base_footprint"/>
+  <joint name="base_footprint_joint" type="fixed"><parent link="base_link"/><child link="base_footprint"/><origin xyz="0 0 ${-(wheel_radius + body_height / 2)}"/></joint>
   <xacro:macro name="drive_wheel" params="name side">
     <link name="${name}_wheel_link">
